Commit message: Added Lidar

File: description/robot.urdf.xacro (robot description, xacro)
@@ -2,4 +2,5 @@
 <robot xmlns:xacro="http://www.ros.org/wiki/xacro"  name="robot">
     <xacro:include filename="robot_core.xacro" />
-    <xacro:include filename="gazebo_control.xacro"/>
+    <xacro:include filename="gazebo_control.xacro" />
+    <xacro:include filename="lidar.xacro" />
 </robot>

File: description/robot_core.xacro (robot description, xacro)
@@ -13,4 +13,7 @@
 	<material name="black">
 		<color rgba="0 0 0 1"/>
+	</material>
+	<material name="red">
+		<color rgba="1 0 0 1"/>
 	</material>
 <!--BASE LINK-->
