Commit message: LIDAR DONE

File: description/lidar.xacro (robot description, xacro)
@@ -3,8 +3,8 @@
     <joint name="laser_joint" type="fixed">
         <parent link="chassis"/>
-        <child link="laser frame"/>
+        <child link="laser_frame"/>
         <origin xyz="0.1 0 0.175" rpy="0 0 0"/>
     </joint>
-    <link name="laser frame">
+    <link name="laser_frame">
 		<visual>
 			<geometry>
@@ -22,6 +22,31 @@
 		</xacro:inertial_cylinder>
 	</link>
-    <gazebo reference="laser frame">
+    <gazebo reference="laser_frame">
 		<material>Gazebo/Red</material>
+		<sensor name="laser" type="ray">
+			<pose> 0 0 0 0 0 0 </pose>
+			<visualize>true</visualize>
+			<update_rate>10</update_rate>
+			<ray>
+				<scan>
+					<horizontal>
+						<samples>360</samples>
+						<min_angle>-3.14</min_angle>
+						<max_angle>3.14</max_angle>
+					</horizontal>
+				</scan>
+				<range>
+					<min>0.3</min>
+					<max>12</max>
+				</range>
+			</ray>
+			<plugin name="laser_controller" filename="libgazebo_ros_ray_sensor.so">
+				<ros>
+					<argument>~/out:=scan</argument>
+				</ros>
+				<output_type>sensor_msgs/LaserScan</output_type>
+				<frame_name>laser_frame</frame_name>
+			</plugin>
+		</sensor>
 	</gazebo>
 </robot>
