Commit message: Added camera sensor

File: description/camera.xacro (robot description, xacro)
@@ -9,7 +9,7 @@
         <visual>
             <geometry>
-                <box size="0.010 0.03 0.03"/>
+               <box size="0.010 0.03 0.03"/>
             </geometry>
-            <material name="red"/>
+            <material name="black"/>
         </visual>
     </link>
@@ -21,5 +21,25 @@
     <link name="camera_link_optical"></link>
     <gazebo reference="camera_link">
-		<material>Gazebo/Red</material>
+		<material>Gazebo/Black</material>
+        <sensor name="camera" type="camera">
+        <pose>0 0 0 0 0 0</pose>
+        <visualize>true</visualize>
+        <update_rate>10</update_rate>
+        <camera>
+            <horizontal_fov>1.089</horizontal_fov>
+            <image>
+                <format>R8G8B8</format>
+                <width>640</width>
+                <height>480</height>
+            </image>
+            <clip>
+                <near>0.05</near>
+                <far>8.0</far>
+            </clip>
+        </camera>
+        <plugin name="camera_controller" filename="libgazebo_ros_camera.so">
+            <frame_name>camera_link_optical</frame_name>
+        </plugin>
+    </sensor>
 	</gazebo>
 </robot>
