Commit message: ADDED GAZEBO CONTROL

File: description/robot_core.xacro (robot description, xacro)
@@ -41,4 +41,7 @@
 		</xacro:inertial_box>
 	</link>
+	<gazebo reference="chassis">
+		<material>Gazebo/White</material>
+	</gazebo>
 	<!--LEFT WHEEL LINK-->
 	<joint name="left_wheel_joint" type="continuous">
@@ -64,4 +67,7 @@
 		</xacro:inertial_cylinder>
 	</link>
+	<gazebo reference="left_wheel">
+		<material>Gazebo/Blue</material>
+	</gazebo>
 	<!--RIGHT WHEEL LINK-->
 	<joint name="right_wheel_joint" type="continuous">
@@ -87,4 +93,7 @@
 		</xacro:inertial_cylinder>
 	</link>
+	<gazebo reference="right_wheel">
+		<material>Gazebo/Blue</material>
+	</gazebo>
 	<!--CASTER WHEEL LINK -->
 	<joint name="caster_wheel_joint" type="fixed">
@@ -109,3 +118,6 @@
 		</xacro:inertial_sphere>
 	</link>
+	<gazebo reference="caster_wheel">
+		<material>Gazebo/Black</material>
+	</gazebo>
 </robot>

Commit message: New

File: description/robot_core.xacro (robot description, xacro)
@@ -20,4 +20,11 @@
 	<link name="base_link">
 	</link>
+	<!--BASE_FOOTPRINT LINK-->
+		<joint name="base_footprint_joint" type="fixed">
+		<parent link="base_link"/>
+		<child link="base_footprint"/>
+		<origin xyz="0 0 0" rpy="0 0 0"/>
+		<link name="base_footprint">
+		</link>
 <!--CHASSIS LINK-->
 	<joint name="chassis_joint" type="fixed">

Commit message: Changes

File: description/robot_core.xacro (robot description, xacro)
@@ -21,10 +21,11 @@
 	</link>
 	<!--BASE_FOOTPRINT LINK-->
-		<joint name="base_footprint_joint" type="fixed">
+	<joint name="base_footprint_joint" type="fixed">
 		<parent link="base_link"/>
 		<child link="base_footprint"/>
 		<origin xyz="0 0 0" rpy="0 0 0"/>
-		<link name="base_footprint">
-		</link>
+	</joint>
+	<link name="base_footprint">
+	</link>
 <!--CHASSIS LINK-->
 	<joint name="chassis_joint" type="fixed">
